Commit message: first commit

File: wsg50_simulation/urdf/wsg50_210.urdf.xacro (robot description, xacro)
@@ -41,9 +41,13 @@
      <limit effort="100" velocity="100"/>
   </joint>
-  <transmission name="${name}_base_trans_left" type="pr2_mechanism_model/SimpleTransmission">
-     <actuator name="${name}_base_motor_left" />
-     <joint name="${name}_base_joint_gripper_left" />
-     <mechanicalReduction>1</mechanicalReduction>
-     <motorTorqueConstant>1</motorTorqueConstant>
+  <transmission name="${name}_base_trans_left">
+     <type>transmission_interface/SimpleTransmission</type>
+     <joint name="${name}_base_joint_gripper_left">
+       <hardwareInterface>hardware_interface/PositionJointInterface</hardwareInterface>
+     </joint>
+     <actuator name="${name}_base_motor_left">
+       <hardwareInterface>hardware_interface/PositionJointInterface</hardwareInterface>
+       <mechanicalReduction>1</mechanicalReduction>
+     </actuator>
   </transmission>
   <link name="${name}_gripper_left">
@@ -126,9 +130,13 @@
      <limit effort="100" velocity="100"/>
   </joint>
-  <transmission name="${name}_base_trans_right" type="pr2_mechanism_model/SimpleTransmission">
-     <actuator name="${name}_base_motor_right" />
-     <joint name="${name}_base_joint_gripper_right" />
-     <mechanicalReduction>1</mechanicalReduction>
-     <motorTorqueConstant>1</motorTorqueConstant>
+  <transmission name="${name}_base_trans_right">
+     <type>transmission_interface/SimpleTransmission</type>
+     <joint name="${name}_base_joint_gripper_right">
+       <hardwareInterface>hardware_interface/PositionJointInterface</hardwareInterface>
+     </joint>
+     <actuator name="${name}_base_motor_right">
+       <hardwareInterface>hardware_interface/PositionJointInterface</hardwareInterface>
+       <mechanicalReduction>1</mechanicalReduction>
+     </actuator>
   </transmission>
     <link name="${name}_gripper_right">

File: wsg50_simulation/urdf/wsg_50.urdf.xacro (robot description, xacro)
@@ -16,7 +16,7 @@
           <mass value="0.25" />
           <origin xyz="0 0 0" />
-     	  <!--inertia ixx="1.0" ixy="0.0" ixz="0.0"
+     	  <inertia ixx="1.0" ixy="0.0" ixz="0.0"
                iyy="100.0" iyz="0.0"
-               izz="1.0" /-->
+               izz="1.0" />
       	  <inertia  ixx="1.0" ixy="0.0"  ixz="0.0"  iyy="1.0"  iyz="0.0"  izz="1.0" />
       </inertial>
@@ -46,5 +46,5 @@
   <joint name="${name}_base_joint_gripper_left" type="prismatic">
      <limit lower="-0.055" upper="-0.0027" effort="1.0" velocity="1.0"/>
-     <origin xyz="0 0 0" rpy="0 0 0" />      <!--origin xyz="-0.0067 0 0.049" rpy="0 0 0" /-->
+     <origin xyz="0 0 0" rpy="0 0 0" />   <!--origin xyz="-0.0067 0 0.049" rpy="0 0 0" /-->
      <parent link="${name}_base_link"/>
      <child link="${name}_gripper_left" />
@@ -53,10 +53,14 @@
      <limit effort="100" velocity="100"/>
   </joint>
-  <transmission name="${name}_base_trans_left" type="pr2_mechanism_model/SimpleTransmission">
-     <actuator name="${name}_base_motor_left" />
-     <joint name="${name}_base_joint_gripper_left" />
-     <mechanicalReduction>1</mechanicalReduction>
-     <motorTorqueConstant>1</motorTorqueConstant>
-  </transmission>
+    <transmission name="${name}_base_trans_left">
+        <type>transmission_interface/SimpleTransmission</type>
+        <joint name="${name}_base_joint_gripper_left">
+            <hardwareInterface>hardware_interface/PositionJointInterface</hardwareInterface>
+        </joint>
+        <actuator name="${name}_base_motor_left">
+            <hardwareInterface>hardware_interface/PositionJointInterface</hardwareInterface>
+            <mechanicalReduction>1</mechanicalReduction>
+        </actuator>
+    </transmission>
   <link name="${name}_gripper_left">
       <inertial>
@@ -73,6 +77,6 @@
 	     <!--box size="0.0175 0.03 0.024"/-->
           </geometry>
-          <material name="black">
-		<color rgba="0 0 0 0"/>
+                    <material name="left_blue">
+                        <color rgba="0.2 0.4 0.9 1"/>
       	  </material>
       </visual>
@@ -112,6 +116,6 @@
              <mesh filename="package://wsg50_simulation/meshes/WSG-FMF.stl" scale="0.001 0.001 0.001"/>
           </geometry>
-          <material name="black">
-		<color rgba="0 0 0 0"/>
+                    <material name="left_blue">
+                <color rgba="0.2 0.4 0.9 1"/>
       	  </material>
       </visual>
@@ -138,10 +142,14 @@
      <limit effort="100" velocity="100"/>
   </joint>
-  <transmission name="${name}_base_trans_right" type="pr2_mechanism_model/SimpleTransmission">
-     <actuator name="${name}_base_motor_right" />
-     <joint name="${name}_base_joint_gripper_right" />
-     <mechanicalReduction>1</mechanicalReduction>
-     <motorTorqueConstant>1</motorTorqueConstant>
-  </transmission>
+    <transmission name="${name}_base_trans_right">
+        <type>transmission_interface/SimpleTransmission</type>
+        <joint name="${name}_base_joint_gripper_right">
+            <hardwareInterface>hardware_interface/PositionJointInterface</hardwareInterface>
+        </joint>
+        <actuator name="${name}_base_motor_right">
+            <hardwareInterface>hardware_interface/PositionJointInterface</hardwareInterface>
+            <mechanicalReduction>1</mechanicalReduction>
+        </actuator>
+    </transmission>
     <link name="${name}_gripper_right">
       <inertial>
@@ -158,18 +166,18 @@
 	     <!--box size="0.0175 0.03 0.024"/-->
           </geometry>
-          <material name="black">
-		<color rgba="0 0 0 0"/>
-      	  </material>
-      </visual>
-      <collision>
-          <origin xyz="0 0 0" rpy="0 0 0" />
-          <geometry>
-	     <!--box size="0.0175 0.03 0.024"/-->
-             <mesh filename="package://wsg50_simulation/meshes/GUIDE_WSG50_110.stl" scale="0.001 0.001 0.001"/>
-         </geometry>
-     </collision>
-     <contact_coefficients kd="1.0" kp="1000.0" mu="0"/>
-  </link>
-  <gazebo reference="gripper_right">
+                    <material name="right_white">
+                <color rgba="1 1 1 1"/>
+      	  </material>
+      </visual>
+      <collision>
+          <origin xyz="0 0 0" rpy="0 0 0" />
+          <geometry>
+	     <!--box size="0.0175 0.03 0.024"/-->
+             <mesh filename="package://wsg50_simulation/meshes/GUIDE_WSG50_110.stl" scale="0.001 0.001 0.001"/>
+         </geometry>
+     </collision>
+     <contact_coefficients kd="1.0" kp="1000.0" mu="0"/>
+  </link>
+    <gazebo reference="${name}_gripper_right">
     <material>Gazebo/White</material>
     <turnGravityOff>false</turnGravityOff>
@@ -197,6 +205,6 @@
              <mesh filename="package://wsg50_simulation/meshes/WSG-FMF.stl" scale="0.001 0.001 0.001"/>
           </geometry>
-          <material name="black">
-		<color rgba="0 0 0 0"/>
+                    <material name="right_white">
+                <color rgba="1 1 1 1"/>
       	  </material>
       </visual>
